File: Laser_CNC.kicad_pcb (KiCad board)
At the start: 2 copper layers, 101.6 x 101.6 mm, 60 parts, among them J1 VCC_24V, J10 Conn_M_PAP_Y, J11 Conn_limit_X, J12 Conn_limit_Y, J13 Conn_limit_Z, J16 Conn_M_PAP_Z, J17 Conn_Laser_OUT, J18 Conn_Laser_OUT, J4 Conn_limit_X, J5 Conn_limit_Y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

Commit message: PCB listo
Parts:
- moved D4 43.6 mm to (176.2, 148.3)
- moved D5 38.8 mm to (173.4, 148.1), turned to 180 degrees
- moved R10 16.9 mm to (174.4, 134.0), turned to -90 degrees
- moved R13 10.5 mm to (170.9, 134.1), turned to -90 degrees
- moved C10 7.47 mm to (172.8, 120.8), turned to 0 degrees
- moved C11 7.39 mm to (173.3, 128.0)
- moved C5 5.03 mm to (126.9, 114.2), turned to 180 degrees
- moved J18 2.94 mm to (144.0, 159.9), turned to 0 degrees
- moved C7 1.46 mm to (142.1, 138.6)
- moved C1 1.45 mm to (127.1, 138.6)
- moved U3 1.45 mm to (136.0, 141.1)
- moved U4 1.45 mm to (120.8, 141.1)
- moved J13 1.22 mm to (153.1, 87.6)
- moved J6 1.22 mm to (145.5, 87.6)
- moved R11 1.22 mm to (164.3, 85.7)
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Connections:
- J11 pad 1: /+5V -> /+5Vdc
- J11 pad 2: /+5V -> /+5Vdc
- J12 pad 1: /+5V -> /+5Vdc
- J12 pad 2: /+5V -> /+5Vdc
- J13 pad 1: /+5V -> /+5Vdc
- J13 pad 2: /+5V -> /+5Vdc
- J4 pad 1: /+5V -> /+5Vdc
- J4 pad 2: /+5V -> /+5Vdc
- J5 pad 1: /+5V -> /+5Vdc
- J5 pad 2: /+5V -> /+5Vdc
- J6 pad 1: /+5V -> /+5Vdc
- J6 pad 2: /+5V -> /+5Vdc
- R11 pad 1: /+5V -> /+5Vdc
- R14 pad 1: /+5V -> /+5Vdc
- R16 pad 1: /+5V -> /+5Vdc
- R17 pad 1: /+5V -> /+5Vdc
- R19 pad 1: /+5V -> /+5Vdc
- R8 pad 1: /+5V -> /+5Vdc
- U1 pad 10: GND -> unconnected-(U1-Pad10)
- U1 pad 9: GND -> unconnected-(U1-Pad9)
- U2 pad 10: GND -> unconnected-(U2-Pad10)
- U2 pad 9: GND -> unconnected-(U2-Pad9)
Routing:
- net /+5Vdc: track 0.00 -> 382.9 mm, vias 0 -> 6
- net GND: track 0.00 -> 132.5 mm, vias 0 -> 10
- net /limit_X: track 4.90 -> 116.9 mm, vias 0 -> 2
- net /step_input_Y: track 0.00 -> 104.2 mm, vias 0 -> 8
- net /limit_Y: track 4.62 -> 93.8 mm, vias 0 -> 2
- net /dir_input_Z: track 0.00 -> 83.8 mm, vias 0 -> 8
- net Net-(U1-Pad11): track 0.00 -> 75.0 mm, vias 0 -> 6
- net Net-(A1-Pad1): track 0.00 -> 71.5 mm, vias 0 -> 2
- net /dir_input_Y: track 0.00 -> 68.4 mm, vias 0 -> 2
- net Net-(U1-Pad6): track 0.00 -> 67.2 mm, vias 0 -> 6
- net /limit_Z: track 5.52 -> 69.5 mm, vias 0 -> 2
- net Net-(A1-Pad2): track 0.00 -> 63.7 mm, vias 0 -> 2
- net /dir_input_X: track 0.00 -> 55.5 mm, vias 0 -> 5
- net /CCW_X: track 0.00 -> 54.2 mm, vias 0 -> 2
- net Net-(U1-Pad3): track 0.00 -> 50.1 mm, vias 0 -> 4
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- added copper zone on B.Cu, net GND
