File: Laser_CNC.kicad_sch (KiCad schematic)
At the start: 66 parts, among them J1 VCC_24V, J10 Conn_M_PAP_Y, J11 Conn_limit_X, J12 Conn_limit_Y, J13 Conn_limit_Z, J14 Conn_L01x02, J15 Conn_01x02, J16 Conn_M_PAP_Z, J17 Conn_Laser_OUT, J18 Conn_Laser_OUT, J2 Conn_01x02, J3 Conn_01x02, J4 Conn_limit_X, J5 Conn_limit_Y, J6 Conn_limit_Z, J7 Conn_M_PAP_X, J8 Conn_01x02, J9 Conn_01x02, Q1 BC548, Q2 BC548, Q3 BC548, U1 74LS00, U2 74LS00, U3 74LS00, U4 74LS04, U5 LM7809_TO220, U6 LM7805_TO220

Commit message: actualizacion
Parts:
- removed J14: Conn_L01x02, symbol Connector_Generic:Conn_01x02
- removed J15, J2, J3, J8, J9: Conn_01x02, symbol Connector_Generic:Conn_01x02
- C1, C10, C3, C5, C7, C9: footprint (none) -> Capacitor_THT:C_Disc_D4.7mm_W2.5mm_P5.00mm
- C11, C8: footprint (none) -> Capacitor_THT:CP_Radial_D10.0mm_P3.50mm
- C2: footprint (none) -> Capacitor_THT:CP_Radial_D13.0mm_P7.50mm
- C4, C6: footprint (none) -> Capacitor_THT:CP_Radial_D13.0mm_P5.00mm
- D3, D4, D5: footprint (none) -> LED_THT:LED_D5.0mm
- F1: footprint (none) -> Fuse:Fuseholder_Cylinder-5x20mm_Stelvio-Kontek_PTF78_Horizontal_Open
- J1: footprint (none) -> TerminalBlock:TerminalBlock_bornier-2_P5.08mm
- J10, J16, J7: footprint (none) -> Connector_Molex:Molex_SL_171971-0012_1x12_P2.54mm_Vertical
- J11, J12, J13, J4, J5, J6: footprint (none) -> Connector_Molex:Molex_SL_171971-0005_1x05_P2.54mm_Vertical
- J17, J18: footprint (none) -> Connector_JST:JST_EH_B2B-EH-A_1x02_P2.50mm_Vertical
- L1: footprint (none) -> Inductor_THT:L_Radial_D6.0mm_P4.00mm
- R1, R10, R11, R12, R13, R14, R15, R16, R17, R18, R19, R2, R3, R4, R5, R6, R7, R8, R9: footprint (none) -> Resistor_THT:R_Axial_DIN0207_L6.3mm_D2.5mm_P10.16mm_Horizontal
- U1, U2, U3, U4: footprint (none) -> Package_DIP:DIP-14_W7.62mm_LongPads
Connections:
- net +5V: no longer R12.1
- net +5Vdc: now also C1.1, C3.1, C5.1, C7.1, C8.1, C9.1, D2.2 (A), R12.1, R5.2, U1.14 (VCC), U2.14 (VCC), U3.14 (VCC), U4.14 (VCC), U6.3 (VO)

Commit message: PCB listo
Connections:
- net +5V: no longer J11.1 (Pin_1), J11.2 (Pin_2), J12.1 (Pin_1), J12.2 (Pin_2), J13.1 (Pin_1), J13.2 (Pin_2), J4.1 (Pin_1), J4.2 (Pin_2), J5.1 (Pin_1), J5.2 (Pin_2), J6.1 (Pin_1), J6.2 (Pin_2), R11.1, R14.1, R16.1, R17.1, R19.1, R8.1
- net +5Vdc: now also J11.1 (Pin_1), J11.2 (Pin_2), J12.1 (Pin_1), J12.2 (Pin_2), J13.1 (Pin_1), J13.2 (Pin_2), J4.1 (Pin_1), J4.2 (Pin_2), J5.1 (Pin_1), J5.2 (Pin_2), J6.1 (Pin_1), J6.2 (Pin_2), R11.1, R14.1, R16.1, R17.1, R19.1, R8.1
- net GND: no longer U1.10, U1.9, U2.10, U2.9
- no-connect marks 22 -> 26
